Commit message: Add files via upload

File: src/myagv_description/urdf/myAGV.urdf (robot description, URDF)
Before this commit: robot myAGV, 2 links, 1 joints
Links:
- removed link base_up
- added link base_link; visual mesh filename=package://myagv_description/meshes/myagv_up.dae scale=1 1 1
Joints:
- joint base_up: child base_up -> base_link
